File: PCBs/PCBs.kicad_sch (KiCad schematic)
At the start: 8 parts, among them P1 Input 1x2, P2 Output 1x2, U1 TPS62172DSGR

Commit message: raspi main compute now
Parts:
- LED1: footprint :LED0805-R-RD -> EasyEDA2KicadFootprints:LED0805-R-RD
Changed lines of the file:
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@@
 			)
 		)
-		(property "Footprint" ":LED0805-R-RD"
+		(property "Footprint" "EasyEDA2KicadFootprints:LED0805-R-RD"
 			(at 163.83 113.03 0)
 			(effects
